Commit message: step 37 of E done

File: body.urdf (robot description, URDF)
Before this commit: robot robot, 1 links, 0 joints
Links:
- removed link Robot
- added link Link0, mass 1; collision box size=1 1 1; visual box size=1 1 1
- added link Link1, mass 1; collision box size=1 1 1; visual box size=1 1 1
- added link Link2, mass 1; collision box size=1 1 1; visual box size=1 1 1
Joints:
- added joint Link0_Link1: type revolute, parent Link0, child Link1, origin xyz=0 0 1.0 rpy=0 0 0, axis 0 1 0, limit lower=-3.14159 upper=3.14159 effort=0.0 velocity=0.0
- added joint Link1_Link2: type revolute, parent Link1, child Link2, origin xyz=0 0 1.0 rpy=0 0 0, axis 0 1 0, limit lower=-3.14159 upper=3.14159 effort=0.0 velocity=0.0

Commit message: finished step E

File: body.urdf (robot description, URDF)
Before this commit: robot robot, 3 links, 2 joints
Links:
- removed link Link0
- removed link Link1
- removed link Link2
- added link BackLeg, mass 1; collision box size=1 1 1; visual box size=1 1 1
- added link FrontLeg, mass 1; collision box size=1 1 1; visual box size=1 1 1
- added link Torso, mass 1; collision box size=1 1 1; visual box size=1 1 1
Joints:
- removed joint Link0_Link1
- removed joint Link1_Link2
- added joint BackLeg_Torso: type revolute, parent BackLeg, child Torso, origin xyz=0 1 1 rpy=0 0 0, axis 0 1 0, limit lower=-3.14159 upper=3.14159 effort=0.0 velocity=0.0
- added joint Torso_FrontLeg: type revolute, parent Torso, child FrontLeg, origin xyz=0 1.0 0 rpy=0 0 0, axis 0 1 0, limit lower=-3.14159 upper=3.14159 effort=0.0 velocity=0.0

Commit message: breh3

File: body.urdf (robot description, URDF)
Before this commit: robot robot, 3 links, 2 joints
Joints:
- removed joint BackLeg_Torso
- added joint Torso_BackLeg: type revolute, parent Torso, child BackLeg, origin xyz=0 1 1 rpy=0 0 0, axis 0 1 0, limit lower=-3.14159 upper=3.14159 effort=0.0 velocity=0.0

Commit message: motors

File: body.urdf (robot description, URDF)
Before this commit: robot robot, 3 links, 2 joints
Joints:
- joint Torso_BackLeg: origin xyz=0 1 1 rpy=0 0 0 -> xyz=0 0.5 1 rpy=0 0 0
- joint Torso_FrontLeg: origin xyz=0 1.0 0 rpy=0 0 0 -> xyz=0 -0.5 1 rpy=0 0 0

Commit message: Revert "motors"
This reverts commit ecc21a5146f85d87f7a209b5eda5253e5362215d.

File: body.urdf (robot description, URDF)
Before this commit: robot robot, 3 links, 2 joints
Joints:
- joint Torso_BackLeg: origin xyz=0 0.5 1 rpy=0 0 0 -> xyz=0 1 1 rpy=0 0 0
- joint Torso_FrontLeg: origin xyz=0 -0.5 1 rpy=0 0 0 -> xyz=0 1.0 0 rpy=0 0 0

Commit message: step 30 of G

File: body.urdf (robot description, URDF)
Before this commit: robot robot, 3 links, 2 joints
Joints:
- joint Torso_BackLeg: origin xyz=0 0.5 1 rpy=0 0 0 -> xyz=0.5 0 1 rpy=0 0 0
- joint Torso_FrontLeg: origin xyz=0 -0.5 1 rpy=0 0 0 -> xyz=-0.5 0 1 rpy=0 0 0

Commit message: assignment 6

File: body.urdf (robot description, URDF)
Before this commit: robot robot, 3 links, 2 joints
Links:
- removed link BackLeg
- removed link FrontLeg
- removed link Torso
Joints:
- removed joint Torso_BackLeg
- removed joint Torso_FrontLeg

Commit message: assignment 6

File: body.urdf (robot description, URDF)
Before this commit: robot robot, 0 links, 0 joints
Links:
- added link Link0, mass 1; collision box size=0.8818574750008688 0.02483008123766972 0.3756951452045145; visual box size=0.8818574750008688 0.02483008123766972 0.3756951452045145
- added link Link1, mass 1; collision box size=0.8948569843994592 0.7027252439312522 0.3718032162604863; visual box size=0.8948569843994592 0.7027252439312522 0.3718032162604863
- added link Link2, mass 1; collision box size=0.7692149274430491 0.6740903497369193 0.25584758333484714; visual box size=0.7692149274430491 0.6740903497369193 0.25584758333484714
- added link Link3, mass 1; collision box size=1.3782022637436087 0.46143225134329247 0.1675152385422264; visual box size=1.3782022637436087 0.46143225134329247 0.1675152385422264
- added link Link4, mass 1; collision box size=1.2062771318485912 0.5393731438937014 0.363138629433289; visual box size=1.2062771318485912 0.5393731438937014 0.363138629433289
- added link Link5, mass 1; collision box size=0.6662056425332333 0.6618752357403057 0.9357790583045521; visual box size=0.6662056425332333 0.6618752357403057 0.9357790583045521
- added link Link6, mass 1; collision box size=0.9790697511224604 0.5477912602532994 0.5623506426673293; visual box size=0.9790697511224604 0.5477912602532994 0.5623506426673293
Joints:
- added joint Link0_Link1: type revolute, parent Link0, child Link1, origin xyz=0.5 0 0.5 rpy=0 0 0, axis 0 1 0, limit lower=-3.14159 upper=3.14159 effort=0.0 velocity=0.0
- added joint Link1_Link2: type revolute, parent Link1, child Link2, origin xyz=1 0 0 rpy=0 0 0, axis 0 1 0, limit lower=-3.14159 upper=3.14159 effort=0.0 velocity=0.0
- added joint Link2_Link3: type revolute, parent Link2, child Link3, origin xyz=1 0 0 rpy=0 0 0, axis 0 1 0, limit lower=-3.14159 upper=3.14159 effort=0.0 velocity=0.0
- added joint Link3_Link4: type revolute, parent Link3, child Link4, origin xyz=1 0 0 rpy=0 0 0, axis 0 1 0, limit lower=-3.14159 upper=3.14159 effort=0.0 velocity=0.0
- added joint Link4_Link5: type revolute, parent Link4, child Link5, origin xyz=1 0 0 rpy=0 0 0, axis 0 1 0, limit lower=-3.14159 upper=3.14159 effort=0.0 velocity=0.0
- added joint Link5_Link6: type revolute, parent Link5, child Link6, origin xyz=1 0 0 rpy=0 0 0, axis 0 1 0, limit lower=-3.14159 upper=3.14159 effort=0.0 velocity=0.0

Commit message: traces of work for assignment 7

File: body.urdf (robot description, URDF)
Before this commit: robot robot, 7 links, 6 joints
Links:
- removed link Link4
- removed link Link5
- removed link Link6
- link Link0: geometry collision box size=1 1 1; visual box size=1 1 1
- link Link1: geometry collision box size=1.1618645523285525 1.3665323187562604 1.122368801570754; visual box size=1.1618645523285525 1.3665323187562604 1.122368801570754
- link Link2: geometry collision box size=0.8232342940896505 1.4829756285249642 1.1172353490736582; visual box size=0.8232342940896505 1.4829756285249642 1.1172353490736582
- link Link3: geometry collision box size=1.3140589751850449 1.211039160185767 1.264497676228313; visual box size=1.3140589751850449 1.211039160185767 1.264497676228313
Joints:
- removed joint Link3_Link4
- removed joint Link4_Link5
- removed joint Link5_Link6
- joint Link0_Link1: origin xyz=0.5 0 0.5 rpy=0 0 0 -> xyz=0 1 0 rpy=0 0 0
- joint Link1_Link2: origin xyz=1 0 0 rpy=0 0 0 -> xyz=0 0 1.1172353490736582 rpy=0 0 0
- joint Link2_Link3: origin xyz=1 0 0 rpy=0 0 0 -> xyz=0 1.211039160185767 0 rpy=0 0 0

Commit message: working assignment 7

File: body.urdf (robot description, URDF)
Before this commit: robot robot, 4 links, 3 joints
Links:
- added link Link4, mass 1; collision box size=0.5284730834731295 2.0834934893822123 1.1854184198755056; visual box size=0.5284730834731295 2.0834934893822123 1.1854184198755056
- added link Link5, mass 1; collision box size=1.9645290984587613 1.776015718432605 1.1067577181312633; visual box size=1.9645290984587613 1.776015718432605 1.1067577181312633
- added link Link6, mass 1; collision box size=1.1604275213494892 2.255871458163117 1.042961228632861; visual box size=1.1604275213494892 2.255871458163117 1.042961228632861
- added link Link7, mass 1; collision box size=1.1287922979676044 1.0812310449997158 1.0676031006525502; visual box size=1.1287922979676044 1.0812310449997158 1.0676031006525502
- link Link0: geometry collision box size=0.5099300681416301 1.9858325745946652 1.4219679122796234; visual box size=0.5099300681416301 1.9858325745946652 1.4219679122796234
- link Link1: geometry collision box size=1.6293718381694324 1.5300173621961333 1.1675770824009721; visual box size=1.6293718381694324 1.5300173621961333 1.1675770824009721
- link Link2: geometry collision box size=0.8630771062800671 1.1479320442751715 1.0165851751973674; visual box size=0.8630771062800671 1.1479320442751715 1.0165851751973674
- link Link3: geometry collision box size=0.8649891498134274 1.2130893034702082 1.0661164571262307; visual box size=0.8649891498134274 1.2130893034702082 1.0661164571262307
Joints:
- removed joint Link0_Link1
- removed joint Link1_Link2
- removed joint Link2_Link3
- added joint Link0_Link3: type revolute, parent Link0, child Link3, origin xyz=0 1.9858325745946652 0 rpy=0 0 0, axis 0 1 0, limit lower=-3.14159 upper=3.14159 effort=0.0 velocity=0.0
- added joint Link1_Link6: type revolute, parent Link1, child Link6, origin xyz=0 -0.7650086810980666 -0.5837885412004861 rpy=0 0 0, axis 0 1 0, limit lower=-3.14159 upper=3.14159 effort=0.0 velocity=0.0
- added joint Link2_Link1: type revolute, parent Link2, child Link1, origin xyz=0.43153855314003353 0 -0.5082925875986837 rpy=0 0 0, axis 0 1 0, limit lower=-3.14159 upper=3.14159 effort=0.0 velocity=0.0
- added joint Link4_Link0: type revolute, parent Link4, child Link0, origin xyz=0.26423654173656475 1.0417467446911062 0 rpy=0 0 0, axis 0 1 0, limit lower=-3.14159 upper=3.14159 effort=0.0 velocity=0.0
- added joint Link5_Link4: type revolute, parent Link5, child Link4, origin xyz=0.9822645492293807 0 -0.5533788590656317 rpy=0 0 0, axis 0 1 0, limit lower=-3.14159 upper=3.14159 effort=0.0 velocity=0.0
- added joint Link6_Link7: type revolute, parent Link6, child Link7, origin xyz=0.5802137606747446 -1.1279357290815586 0 rpy=0 0 0, axis 0 1 0, limit lower=-3.14159 upper=3.14159 effort=0.0 velocity=0.0
- added joint Link7_Link5: type revolute, parent Link7, child Link5, origin xyz=0.5643961489838022 0 -0.5338015503262751 rpy=0 0 0, axis 0 1 0, limit lower=-3.14159 upper=3.14159 effort=0.0 velocity=0.0

Commit message: Assignment 7

File: body.urdf (robot description, URDF)
Before this commit: robot robot, 8 links, 7 joints
Links:
- added link Link10, mass 1; collision box size=0.6463908104208413 1.6752384803764986 1.4393205507006384; visual box size=0.6463908104208413 1.6752384803764986 1.4393205507006384
- added link Link11, mass 1; collision box size=1.4534215124192005 1.2187475614581225 1.2490636113925517; visual box size=1.4534215124192005 1.2187475614581225 1.2490636113925517
- added link Link12, mass 1; collision box size=1.0622338880248883 1.877154794003474 1.1728944575095146; visual box size=1.0622338880248883 1.877154794003474 1.1728944575095146
- added link Link8, mass 1; collision box size=1.6163906389820952 1.1512050644843344 1.3601361779348116; visual box size=1.6163906389820952 1.1512050644843344 1.3601361779348116
- added link Link9, mass 1; collision box size=1.2519341799775319 1.8848488809410497 1.1783089243502114; visual box size=1.2519341799775319 1.8848488809410497 1.1783089243502114
- link Link0: geometry collision box size=1.4416364677796705 1.7978791244575838 1.022365996345513; visual box size=1.4416364677796705 1.7978791244575838 1.022365996345513
- link Link1: geometry collision box size=1.8756000415252134 2.2685707861108027 1.3863881564940388; visual box size=1.8756000415252134 2.2685707861108027 1.3863881564940388
- link Link2: geometry collision box size=0.5944851543157041 1.5216022043442932 1.3603684383435992; visual box size=0.5944851543157041 1.5216022043442932 1.3603684383435992
- link Link3: geometry collision box size=0.6528224122324835 1.664485245812995 1.144387082367152; visual box size=0.6528224122324835 1.664485245812995 1.144387082367152
- link Link4: geometry collision box size=1.3184639807084286 1.7880154529664882 1.1314797969288515; visual box size=1.3184639807084286 1.7880154529664882 1.1314797969288515
- link Link5: geometry collision box size=1.4479375080494021 1.5882451176895651 1.4503639881564505; visual box size=1.4479375080494021 1.5882451176895651 1.4503639881564505
- link Link6: geometry collision box size=1.1531879483490337 1.9707804904295902 1.2084274510593773; visual box size=1.1531879483490337 1.9707804904295902 1.2084274510593773
- link Link7: geometry collision box size=1.1109277882026447 1.6015497137262416 1.1121514652101216; visual box size=1.1109277882026447 1.6015497137262416 1.1121514652101216
Joints:
- removed joint Link0_Link3
- removed joint Link1_Link6
- removed joint Link2_Link1
- removed joint Link4_Link0
- removed joint Link5_Link4
- removed joint Link6_Link7
- removed joint Link7_Link5
- added joint Link0_Link5: type revolute, parent Link0, child Link5, origin xyz=0 -1.7978791244575838 0 rpy=0 0 0, axis 0 1 0, limit lower=-3.14159 upper=3.14159 effort=0.0 velocity=0.0
- added joint Link10_Link11: type revolute, parent Link10, child Link11, origin xyz=0 0.8376192401882493 0.7196602753503192 rpy=0 0 0, axis 0 1 0, limit lower=-3.14159 upper=3.14159 effort=0.0 velocity=0.0
- added joint Link11_Link8: type revolute, parent Link11, child Link8, origin xyz=0.7267107562096002 0.6093737807290612 0 rpy=0 0 0, axis 0 1 0, limit lower=-3.14159 upper=3.14159 effort=0.0 velocity=0.0
- added joint Link12_Link7: type revolute, parent Link12, child Link7, origin xyz=1.0622338880248883 0 0 rpy=0 0 0, axis 0 1 0, limit lower=-3.14159 upper=3.14159 effort=0.0 velocity=0.0
- added joint Link1_Link0: type revolute, parent Link1, child Link0, origin xyz=0 -1.1342853930554013 -0.6931940782470194 rpy=0 0 0, axis 0 1 0, limit lower=-3.14159 upper=3.14159 effort=0.0 velocity=0.0
- added joint Link3_Link2: type revolute, parent Link3, child Link2, origin xyz=0.32641120611624175 0.8322426229064975 0 rpy=0 0 0, axis 0 1 0, limit lower=-3.14159 upper=3.14159 effort=0.0 velocity=0.0
- added joint Link4_Link6: type revolute, parent Link4, child Link6, origin xyz=0 0 -1.1314797969288515 rpy=0 0 0, axis 0 1 0, limit lower=-3.14159 upper=3.14159 effort=0.0 velocity=0.0
- added joint Link5_Link9: type revolute, parent Link5, child Link9, origin xyz=0.7239687540247011 -0.7941225588447826 0 rpy=0 0 0, axis 0 1 0, limit lower=-3.14159 upper=3.14159 effort=0.0 velocity=0.0
- added joint Link6_Link1: type revolute, parent Link6, child Link1, origin xyz=0 0 -1.2084274510593773 rpy=0 0 0, axis 0 1 0, limit lower=-3.14159 upper=3.14159 effort=0.0 velocity=0.0
- added joint Link7_Link10: type revolute, parent Link7, child Link10, origin xyz=0.5554638941013224 0 0.5560757326050608 rpy=0 0 0, axis 0 1 0, limit lower=-3.14159 upper=3.14159 effort=0.0 velocity=0.0
- added joint Link8_Link4: type revolute, parent Link8, child Link4, origin xyz=0.8081953194910476 0 -0.6800680889674058 rpy=0 0 0, axis 0 1 0, limit lower=-3.14159 upper=3.14159 effort=0.0 velocity=0.0
- added joint Link9_Link3: type revolute, parent Link9, child Link3, origin xyz=1.2519341799775319 0 0 rpy=0 0 0, axis 0 1 0, limit lower=-3.14159 upper=3.14159 effort=0.0 velocity=0.0

Commit message: new base quadruped code

File: body.urdf (robot description, URDF)
Before this commit: robot robot, 7 links, 6 joints
Links:
- removed link Link0
- removed link Link1
- removed link Link2
- removed link Link3
- removed link Link4
- removed link Link5
- removed link Link6
- added link BackLeg, mass 1; collision box size=0.2 1 0.2; visual box size=0.2 1 0.2
- added link BackLowerLeg, mass 1; collision box size=0.2 0.2 1; visual box size=0.2 0.2 1
- added link FrontLeg, mass 1; collision box size=0.2 1 0.2; visual box size=0.2 1 0.2
- added link FrontLowerLeg, mass 1; collision box size=0.2 0.2 1; visual box size=0.2 0.2 1
- added link LeftLeg, mass 1; collision box size=1 0.2 0.2; visual box size=1 0.2 0.2
- added link LeftLowerLeg, mass 1; collision box size=0.2 0.2 1; visual box size=0.2 0.2 1
- added link RightLeg, mass 1; collision box size=1 0.2 0.2; visual box size=1 0.2 0.2
- added link RightLowerLeg, mass 1; collision box size=0.2 0.2 1; visual box size=0.2 0.2 1
- added link Torso, mass 1; collision box size=1 1 1; visual box size=1 1 1
Joints:
- removed joint Link0_Link1
- removed joint Link1_Link2
- removed joint Link2_Link3
- removed joint Link3_Link4
- removed joint Link4_Link5
- removed joint Link5_Link6
- added joint BackLeg_BackLowerLeg: type revolute, parent BackLeg, child BackLowerLeg, origin xyz=0 -1 0 rpy=0 0 0, axis 1 0 0, limit lower=-3.14159 upper=3.14159 effort=0.0 velocity=0.0
- added joint FrontLeg_FrontLowerLeg: type revolute, parent FrontLeg, child FrontLowerLeg, origin xyz=0 1 0 rpy=0 0 0, axis 1 0 0, limit lower=-3.14159 upper=3.14159 effort=0.0 velocity=0.0
- added joint LeftLeg_LeftLowerLeg: type revolute, parent LeftLeg, child LeftLowerLeg, origin xyz=-1 0 0 rpy=0 0 0, axis 0 1 0, limit lower=-3.14159 upper=3.14159 effort=0.0 velocity=0.0
- added joint RightLeg_RightLowerLeg: type revolute, parent RightLeg, child RightLowerLeg, origin xyz=1 0 0 rpy=0 0 0, axis 0 1 0, limit lower=-3.14159 upper=3.14159 effort=0.0 velocity=0.0
- added joint Torso_BackLeg: type revolute, parent Torso, child BackLeg, origin xyz=0 -0.5 1 rpy=0 0 0, axis 1 0 0, limit lower=-3.14159 upper=3.14159 effort=0.0 velocity=0.0
- added joint Torso_FrontLeg: type revolute, parent Torso, child FrontLeg, origin xyz=0 0.5 1 rpy=0 0 0, axis 1 0 0, limit lower=-3.14159 upper=3.14159 effort=0.0 velocity=0.0
- added joint Torso_LeftLeg: type revolute, parent Torso, child LeftLeg, origin xyz=-0.5 0 1 rpy=0 0 0, axis 0 1 0, limit lower=-3.14159 upper=3.14159 effort=0.0 velocity=0.0
- added joint Torso_RightLeg: type revolute, parent Torso, child RightLeg, origin xyz=0.5 0 1 rpy=0 0 0, axis 0 1 0, limit lower=-3.14159 upper=3.14159 effort=0.0 velocity=0.0

Commit message: need to edit links

File: body.urdf (robot description, URDF)
Before this commit: robot robot, 9 links, 8 joints
Links:
- added link BottomLeg, mass 1; collision box size=0.6058709658991894 0.024391505721787166 0.580182953613601; visual box size=0.6058709658991894 0.024391505721787166 0.580182953613601
- added link TopLeg, mass 1; collision box size=0.708604931649435 0.9120906259813597 0.9231791186649696; visual box size=0.708604931649435 0.9120906259813597 0.9231791186649696
- link BackLeg: geometry collision box size=1.3709816590900985 0.9947903050698721 0.6780073457504502; visual box size=1.3709816590900985 0.9947903050698721 0.6780073457504502
- link FrontLeg: geometry collision box size=0.5729985074317645 0.6379903484131959 0.891869483124698; visual box size=0.5729985074317645 0.6379903484131959 0.891869483124698
- link LeftLeg: geometry collision box size=1.2549454354688683 0.635636485651113 0.7709991169171602; visual box size=1.2549454354688683 0.635636485651113 0.7709991169171602
- link RightLeg: geometry collision box size=0.7287297166867441 0.4826808161427286 0.4876021967350078; visual box size=0.7287297166867441 0.4826808161427286 0.4876021967350078
Joints:
- added joint Torso_BottomLeg: type revolute, parent Torso, child BottomLeg, origin xyz=0 0 0.5 rpy=0 0 0, axis 0 0 1, limit lower=-3.14159 upper=3.14159 effort=0.0 velocity=0.0
- added joint Torso_TopLeg: type revolute, parent Torso, child TopLeg, origin xyz=0 0 1.5 rpy=0 0 0, axis 0 0 1, limit lower=-3.14159 upper=3.14159 effort=0.0 velocity=0.0

Commit message: almost done

File: body.urdf (robot description, URDF)
Before this commit: robot robot, 11 links, 10 joints
Links:
- removed link BackLeg
- removed link BackLowerLeg
- removed link BottomLeg
- removed link FrontLeg
- removed link FrontLowerLeg
- removed link LeftLeg
- removed link LeftLowerLeg
- removed link RightLeg
- removed link RightLowerLeg
- removed link TopLeg
- removed link Torso
- added link Link0, mass 1; collision box size=1 1 1; visual box size=1 1 1
- added link Link1, mass 1; collision box size=1.039969245077808 0.9560463820239767 1.1351279301823745; visual box size=1.039969245077808 0.9560463820239767 1.1351279301823745
- added link Link2, mass 1; collision box size=0.7522350252240322 0.971518733108805 1.4712481877065304; visual box size=0.7522350252240322 0.971518733108805 1.4712481877065304
- added link Link3, mass 1; collision box size=1.4891256497279601 1.237166854364851 1.22964036732662; visual box size=1.4891256497279601 1.237166854364851 1.22964036732662
- added link Link4, mass 1; collision box size=1.2098694644702697 0.8006208285100241 0.6739398713472199; visual box size=1.2098694644702697 0.8006208285100241 0.6739398713472199
- added link Link5, mass 1; collision box size=0.588953651939706 1.3959868107793172 1.2603647182355828; visual box size=0.588953651939706 1.3959868107793172 1.2603647182355828
- added link Link6, mass 1; collision box size=1.3552211778947871 1.01623133106906 0.7590402927656044; visual box size=1.3552211778947871 1.01623133106906 0.7590402927656044
- added link Link7, mass 1; collision box size=1.26527950535477 1.0715445417604361 1.1887900531137134; visual box size=1.26527950535477 1.0715445417604361 1.1887900531137134
Joints:
- removed joint BackLeg_BackLowerLeg
- removed joint FrontLeg_FrontLowerLeg
- removed joint LeftLeg_LeftLowerLeg
- removed joint RightLeg_RightLowerLeg
- removed joint Torso_BackLeg
- removed joint Torso_BottomLeg
- removed joint Torso_FrontLeg
- removed joint Torso_LeftLeg
- removed joint Torso_RightLeg
- removed joint Torso_TopLeg
- added joint Link0_Link1: type revolute, parent Link0, child Link1, origin xyz=1.1053704645383022 1.1919778194714301 0.30058413554721836 rpy=0 0 0, axis 0 0 1, limit lower=-3.14159 upper=3.14159 effort=0.0 velocity=0.0
- added joint Link0_Link2: type revolute, parent Link0, child Link2, origin xyz=0.5526852322691511 1.1919778194714301 0.6011682710944367 rpy=0 0 0, axis 0 1 0, limit lower=-3.14159 upper=3.14159 effort=0.0 velocity=0.0
- added joint Link0_Link3: type revolute, parent Link0, child Link3, origin xyz=-0.5526852322691511 1.1919778194714301 0.6011682710944367 rpy=0 0 0, axis 0 1 0, limit lower=-3.14159 upper=3.14159 effort=0.0 velocity=0.0
- added joint Link0_Link4: type revolute, parent Link0, child Link4, origin xyz=1.1053704645383022 1.1919778194714301 -0.30058413554721836 rpy=0 0 0, axis 0 0 1, limit lower=-3.14159 upper=3.14159 effort=0.0 velocity=0.0
- added joint Link0_Link6: type revolute, parent Link0, child Link6, origin xyz=1.1053704645383022 -0.5959889097357151 0.6011682710944367 rpy=0 0 0, axis 1 0 0, limit lower=-3.14159 upper=3.14159 effort=0.0 velocity=0.0
- added joint Link0_Link7: type revolute, parent Link0, child Link7, origin xyz=1.1053704645383022 1.1919778194714301 -0.30058413554721836 rpy=0 0 0, axis 0 0 1, limit lower=-3.14159 upper=3.14159 effort=0.0 velocity=0.0
- added joint Link4_Link5: type revolute, parent Link4, child Link5, origin xyz=1.2098694644702697 0.40031041425501207 0.6739398713472199 rpy=0 0 0, axis 1 0 0, limit lower=-3.14159 upper=3.14159 effort=0.0 velocity=0.0
