Commit message: finished revised assignment 7

File: body.urdf (robot description, URDF)
Before this commit: robot robot, 8 links, 7 joints
Links:
- removed link Link1
- removed link Link2
- removed link Link3
- removed link Link4
- removed link Link5
- removed link Link6
- removed link Link7
Joints:
- removed joint Link0_Link2
- removed joint Link0_Link6
- removed joint Link0_Link7
- removed joint Link4_Link5
- added joint Link1_Link2: type revolute, parent Link1, child Link2, origin xyz=-0.5779565697003803 0 0 rpy=0 0 0, axis 0 1 0, limit lower=-3.14159 upper=3.14159 effort=0.0 velocity=0.0
- added joint Link1_Link5: type revolute, parent Link1, child Link5, origin xyz=0 0 -0.2556979051362442 rpy=0 0 0, axis 0 0 1, limit lower=-3.14159 upper=3.14159 effort=0.0 velocity=0.0
- added joint Link5_Link6: type revolute, parent Link5, child Link6, origin xyz=0 -0.40979003537354614 0 rpy=0 0 0, axis 1 0 0, limit lower=-3.14159 upper=3.14159 effort=0.0 velocity=0.0
- added joint Link5_Link7: type revolute, parent Link5, child Link7, origin xyz=0 -0.40979003537354614 0 rpy=0 0 0, axis 1 0 0, limit lower=-3.14159 upper=3.14159 effort=0.0 velocity=0.0
- joint Link0_Link1: axis 0 0 1 -> 1 0 0; origin xyz=1.1053704645383022 1.1919778194714301 0.30058413554721836 rpy=0 0 0 -> xyz=0 0.5 1 rpy=0 0 0
- joint Link0_Link3: origin xyz=-0.5526852322691511 1.1919778194714301 0.6011682710944367 rpy=0 0 0 -> xyz=0.5 0 1 rpy=0 0 0
- joint Link0_Link4: origin xyz=1.1053704645383022 1.1919778194714301 -0.30058413554721836 rpy=0 0 0 -> xyz=0 0 1.5 rpy=0 0 0
