Commit message: hillclimbing creature that mutates brain

File: body0.urdf (robot description, URDF)
Before this commit: robot robot, 8 links, 7 joints
Links:
- removed link Link7
- link Link1: geometry collision box size=1.0300500205474097 0.355542481564197 0.30718710584552433; visual box size=1.0300500205474097 0.355542481564197 0.30718710584552433
- link Link2: geometry collision box size=0.3832624188871543 0.6880671121345705 0.2467496158522661; visual box size=0.3832624188871543 0.6880671121345705 0.2467496158522661
- link Link3: geometry collision box size=1.0860931860959793 0.539760761506236 0.13926722002104155; visual box size=1.0860931860959793 0.539760761506236 0.13926722002104155
- link Link4: geometry collision box size=0.5756503853929865 0.3581853152086615 0.9841506322255935; visual box size=0.5756503853929865 0.3581853152086615 0.9841506322255935
- link Link5: geometry collision box size=0.3252517545403715 0.2610714499540082 0.9513293437884611; visual box size=0.3252517545403715 0.2610714499540082 0.9513293437884611
- link Link6: geometry collision box size=1.086372245975308 0.8843141263775022 0.7382860148868748; visual box size=1.086372245975308 0.8843141263775022 0.7382860148868748
Joints:
- removed joint Link0_Link2
- removed joint Link0_Link5
- removed joint Link1_Link3
- removed joint Link1_Link4
- removed joint Link2_Link7
- removed joint Link3_Link6
- added joint Link0_Link3: type revolute, parent Link0, child Link3, origin xyz=0.5 0 1 rpy=0 0 0, axis 0 1 0, limit lower=-3.14159 upper=3.14159 effort=0.0 velocity=0.0
- added joint Link1_Link2: type revolute, parent Link1, child Link2, origin xyz=0 -0.1777712407820985 0 rpy=0 0 0, axis 1 0 0, limit lower=-3.14159 upper=3.14159 effort=0.0 velocity=0.0
- added joint Link1_Link5: type revolute, parent Link1, child Link5, origin xyz=0 -0.1777712407820985 0 rpy=0 0 0, axis 1 0 0, limit lower=-3.14159 upper=3.14159 effort=0.0 velocity=0.0
- added joint Link2_Link4: type revolute, parent Link2, child Link4, origin xyz=0 0.6880671121345705 0 rpy=0 0 0, axis 1 0 0, limit lower=-3.14159 upper=3.14159 effort=0.0 velocity=0.0
- added joint Link4_Link6: type revolute, parent Link4, child Link6, origin xyz=0 -0.17909265760433074 0 rpy=0 0 0, axis 1 0 0, limit lower=-3.14159 upper=3.14159 effort=0.0 velocity=0.0
- joint Link0_Link1: axis 0 1 0 -> 1 0 0; origin xyz=0.5 0 1 rpy=0 0 0 -> xyz=0 0.5 1 rpy=0 0 0

File: body1.urdf (robot description, URDF)
Before this commit: robot robot, 5 links, 4 joints
Links:
- added link Link5, mass 1; collision box size=0.21909408745712214 0.48928092413710966 0.3526777319034543; visual box size=0.21909408745712214 0.48928092413710966 0.3526777319034543
- added link Link6, mass 1; collision box size=0.6965865639343479 0.2601288850698773 0.9161160361307602; visual box size=0.6965865639343479 0.2601288850698773 0.9161160361307602
- added link Link7, mass 1; collision box size=0.70589245684393 0.5901368284682497 0.1813332933764004; visual box size=0.70589245684393 0.5901368284682497 0.1813332933764004
- link Link1: geometry collision box size=0.8153165213336812 1.0431142960911555 0.12766995280502216; visual box size=0.8153165213336812 1.0431142960911555 0.12766995280502216
- link Link2: geometry collision box size=0.8600618143328433 0.8293267693940193 0.9678578064494086; visual box size=0.8600618143328433 0.8293267693940193 0.9678578064494086
- link Link3: geometry collision box size=0.6330203075163148 0.48185380233716013 0.13291348360948543; visual box size=0.6330203075163148 0.48185380233716013 0.13291348360948543
- link Link4: geometry collision box size=0.6256443572027992 0.8421034346280386 0.6070166750685325; visual box size=0.6256443572027992 0.8421034346280386 0.6070166750685325
Joints:
- removed joint Link0_Link4
- added joint Link0_Link6: type revolute, parent Link0, child Link6, origin xyz=0 0 0.5 rpy=0 0 0, axis 0 0 1, limit lower=-3.14159 upper=3.14159 effort=0.0 velocity=0.0
- added joint Link3_Link4: type revolute, parent Link3, child Link4, origin xyz=0 0.48185380233716013 0 rpy=0 0 0, axis 1 0 0, limit lower=-3.14159 upper=3.14159 effort=0.0 velocity=0.0
- added joint Link4_Link5: type revolute, parent Link4, child Link5, origin xyz=0.6256443572027992 0 0 rpy=0 0 0, axis 0 1 0, limit lower=-3.14159 upper=3.14159 effort=0.0 velocity=0.0
- added joint Link4_Link7: type revolute, parent Link4, child Link7, origin xyz=0 -0.4210517173140193 0 rpy=0 0 0, axis 1 0 0, limit lower=-3.14159 upper=3.14159 effort=0.0 velocity=0.0
- joint Link0_Link1: axis 0 1 0 -> 1 0 0; origin xyz=0.5 0 1 rpy=0 0 0 -> xyz=0 0.5 1 rpy=0 0 0
- joint Link0_Link2: axis 0 1 0 -> 1 0 0; origin xyz=0.5 0 1 rpy=0 0 0 -> xyz=0 0.5 1 rpy=0 0 0
- joint Link2_Link3: axis 0 1 0 -> 1 0 0; origin xyz=-0.20276280435856134 0 0 rpy=0 0 0 -> xyz=0 -0.41466338469700964 0 rpy=0 0 0

File: body2.urdf (robot description, URDF)
Before this commit: robot robot, 5 links, 4 joints
Links:
- added link Link5, mass 1; collision box size=0.6717473258068808 0.9392822622987711 0.2100168719993796; visual box size=0.6717473258068808 0.9392822622987711 0.2100168719993796
- added link Link6, mass 1; collision box size=0.12494974408883155 0.9465490839307625 0.4335407364864792; visual box size=0.12494974408883155 0.9465490839307625 0.4335407364864792
- link Link1: geometry collision box size=0.7581225952937569 0.5334572816580214 0.4158284206448998; visual box size=0.7581225952937569 0.5334572816580214 0.4158284206448998
- link Link2: geometry collision box size=0.6470773191447883 0.9533962707001292 0.26870776421091835; visual box size=0.6470773191447883 0.9533962707001292 0.26870776421091835
- link Link3: geometry collision box size=0.6576919575772031 0.482913586546702 0.8055789418038266; visual box size=0.6576919575772031 0.482913586546702 0.8055789418038266
- link Link4: geometry collision box size=0.540949712924473 0.36954083663878967 0.30366073393483195; visual box size=0.540949712924473 0.36954083663878967 0.30366073393483195
Joints:
- removed joint Link1_Link2
- removed joint Link2_Link4
- added joint Link0_Link2: type revolute, parent Link0, child Link2, origin xyz=0 0 1.5 rpy=0 0 0, axis 0 0 1, limit lower=-3.14159 upper=3.14159 effort=0.0 velocity=0.0
- added joint Link0_Link6: type revolute, parent Link0, child Link6, origin xyz=0 -0.5 1 rpy=0 0 0, axis 1 0 0, limit lower=-3.14159 upper=3.14159 effort=0.0 velocity=0.0
- added joint Link1_Link4: type revolute, parent Link1, child Link4, origin xyz=0 0 0.2079142103224499 rpy=0 0 0, axis 0 0 1, limit lower=-3.14159 upper=3.14159 effort=0.0 velocity=0.0
- added joint Link1_Link5: type revolute, parent Link1, child Link5, origin xyz=0 0.5334572816580214 0 rpy=0 0 0, axis 1 0 0, limit lower=-3.14159 upper=3.14159 effort=0.0 velocity=0.0
- joint Link1_Link3: axis 0 0 1 -> 0 1 0; origin xyz=0 0 -0.5157212829956332 rpy=0 0 0 -> xyz=-0.7581225952937569 0 0 rpy=0 0 0

File: body3.urdf (robot description, URDF)
Before this commit: robot robot, 4 links, 3 joints
Links:
- added link Link4, mass 1; collision box size=0.4897814639964124 1.0309561813026746 0.2241574684293636; visual box size=0.4897814639964124 1.0309561813026746 0.2241574684293636
- added link Link5, mass 1; collision box size=1.043944129687256 0.5188515606584863 0.48223452618878904; visual box size=1.043944129687256 0.5188515606584863 0.48223452618878904
- added link Link6, mass 1; collision box size=0.17989275554139886 0.691933858496368 0.17280745799790356; visual box size=0.17989275554139886 0.691933858496368 0.17280745799790356
- added link Link7, mass 1; collision box size=0.45549226736152193 0.658911978719478 0.9610509063492852; visual box size=0.45549226736152193 0.658911978719478 0.9610509063492852
- link Link1: geometry collision box size=0.418754921383494 0.4535787424720895 0.6443214550381721; visual box size=0.418754921383494 0.4535787424720895 0.6443214550381721
- link Link2: geometry collision box size=0.37662331894193923 0.7157448671956707 0.18899039457002045; visual box size=0.37662331894193923 0.7157448671956707 0.18899039457002045
- link Link3: geometry collision box size=0.9901363288852127 1.035055780942857 0.22101429503811745; visual box size=0.9901363288852127 1.035055780942857 0.22101429503811745
Joints:
- added joint Link2_Link6: type revolute, parent Link2, child Link6, origin xyz=0 0.7157448671956707 0 rpy=0 0 0, axis 1 0 0, limit lower=-3.14159 upper=3.14159 effort=0.0 velocity=0.0
- added joint Link3_Link4: type revolute, parent Link3, child Link4, origin xyz=0 1.035055780942857 0 rpy=0 0 0, axis 1 0 0, limit lower=-3.14159 upper=3.14159 effort=0.0 velocity=0.0
- added joint Link3_Link5: type revolute, parent Link3, child Link5, origin xyz=0 0 -0.11050714751905873 rpy=0 0 0, axis 0 0 1, limit lower=-3.14159 upper=3.14159 effort=0.0 velocity=0.0
- added joint Link6_Link7: type revolute, parent Link6, child Link7, origin xyz=0 0.691933858496368 0 rpy=0 0 0, axis 1 0 0, limit lower=-3.14159 upper=3.14159 effort=0.0 velocity=0.0
- joint Link0_Link1: axis 0 1 0 -> 0 0 1; origin xyz=-0.5 0 1 rpy=0 0 0 -> xyz=0 0 1.5 rpy=0 0 0
- joint Link1_Link2: axis 0 1 0 -> 0 0 1; origin xyz=0.23909862452316236 0 0 rpy=0 0 0 -> xyz=0 0 -0.32216072751908603 rpy=0 0 0
- joint Link1_Link3: origin xyz=0.23909862452316236 0 0 rpy=0 0 0 -> xyz=0.418754921383494 0 0 rpy=0 0 0

File: body4.urdf (robot description, URDF)
Before this commit: robot robot, 8 links, 7 joints
Links:
- removed link Link6
- removed link Link7
- link Link1: geometry collision box size=0.648500844201073 0.336504335942426 0.1768324977179835; visual box size=0.648500844201073 0.336504335942426 0.1768324977179835
- link Link2: geometry collision box size=1.0135407297609595 0.3661030640650461 0.42166310260487194; visual box size=1.0135407297609595 0.3661030640650461 0.42166310260487194
- link Link3: geometry collision box size=0.3857095506151792 0.4733346587691296 0.726226126595371; visual box size=0.3857095506151792 0.4733346587691296 0.726226126595371
- link Link4: geometry collision box size=0.1711014253315231 0.16586437433646664 0.8443779112033238; visual box size=0.1711014253315231 0.16586437433646664 0.8443779112033238
- link Link5: geometry collision box size=0.8124675875953125 0.6154785553284724 0.5423136928231626; visual box size=0.8124675875953125 0.6154785553284724 0.5423136928231626
Joints:
- removed joint Link1_Link3
- removed joint Link2_Link5
- removed joint Link2_Link7
- removed joint Link4_Link6
- added joint Link0_Link3: type revolute, parent Link0, child Link3, origin xyz=0 0 1.5 rpy=0 0 0, axis 0 0 1, limit lower=-3.14159 upper=3.14159 effort=0.0 velocity=0.0
- added joint Link0_Link5: type revolute, parent Link0, child Link5, origin xyz=0.5 0 1 rpy=0 0 0, axis 0 1 0, limit lower=-3.14159 upper=3.14159 effort=0.0 velocity=0.0
- joint Link0_Link1: axis 0 0 1 -> 0 1 0; origin xyz=0 0 0.5 rpy=0 0 0 -> xyz=0.5 0 1 rpy=0 0 0
- joint Link2_Link4: origin xyz=0.9646138679211316 0 0 rpy=0 0 0 -> xyz=-1.0135407297609595 0 0 rpy=0 0 0

File: body5.urdf (robot description, URDF)
Before this commit: robot robot, 8 links, 7 joints
Links:
- removed link Link7
- link Link1: geometry collision box size=1.0300500205474097 0.355542481564197 0.30718710584552433; visual box size=1.0300500205474097 0.355542481564197 0.30718710584552433
- link Link2: geometry collision box size=0.3832624188871543 0.6880671121345705 0.2467496158522661; visual box size=0.3832624188871543 0.6880671121345705 0.2467496158522661
- link Link3: geometry collision box size=1.0860931860959793 0.539760761506236 0.13926722002104155; visual box size=1.0860931860959793 0.539760761506236 0.13926722002104155
- link Link4: geometry collision box size=0.5756503853929865 0.3581853152086615 0.9841506322255935; visual box size=0.5756503853929865 0.3581853152086615 0.9841506322255935
- link Link5: geometry collision box size=0.3252517545403715 0.2610714499540082 0.9513293437884611; visual box size=0.3252517545403715 0.2610714499540082 0.9513293437884611
- link Link6: geometry collision box size=1.086372245975308 0.8843141263775022 0.7382860148868748; visual box size=1.086372245975308 0.8843141263775022 0.7382860148868748
Joints:
- removed joint Link0_Link4
- removed joint Link0_Link5
- removed joint Link1_Link3
- removed joint Link1_Link6
- removed joint Link6_Link7
- added joint Link0_Link3: type revolute, parent Link0, child Link3, origin xyz=0 0.5 1 rpy=0 0 0, axis 1 0 0, limit lower=-3.14159 upper=3.14159 effort=0.0 velocity=0.0
- added joint Link1_Link5: type revolute, parent Link1, child Link5, origin xyz=0 -0.1777712407820985 0 rpy=0 0 0, axis 1 0 0, limit lower=-3.14159 upper=3.14159 effort=0.0 velocity=0.0
- added joint Link2_Link4: type revolute, parent Link2, child Link4, origin xyz=0 0 0.12337480792613305 rpy=0 0 0, axis 0 0 1, limit lower=-3.14159 upper=3.14159 effort=0.0 velocity=0.0
- added joint Link4_Link6: type revolute, parent Link4, child Link6, origin xyz=0 0.3581853152086615 0 rpy=0 0 0, axis 1 0 0, limit lower=-3.14159 upper=3.14159 effort=0.0 velocity=0.0
- joint Link0_Link1: axis 0 0 1 -> 0 1 0; origin xyz=0 0 1.5 rpy=0 0 0 -> xyz=0.5 0 1 rpy=0 0 0
- joint Link1_Link2: axis 0 1 0 -> 0 0 1; origin xyz=1.079560291847085 0 0 rpy=0 0 0 -> xyz=0 0 0.15359355292276217 rpy=0 0 0

File: body6.urdf (robot description, URDF)
Before this commit: robot robot, 5 links, 4 joints
Links:
- added link Link5, mass 1; collision box size=0.21909408745712214 0.48928092413710966 0.3526777319034543; visual box size=0.21909408745712214 0.48928092413710966 0.3526777319034543
- added link Link6, mass 1; collision box size=0.6965865639343479 0.2601288850698773 0.9161160361307602; visual box size=0.6965865639343479 0.2601288850698773 0.9161160361307602
- added link Link7, mass 1; collision box size=0.70589245684393 0.5901368284682497 0.1813332933764004; visual box size=0.70589245684393 0.5901368284682497 0.1813332933764004
- link Link1: geometry collision box size=0.8153165213336812 1.0431142960911555 0.12766995280502216; visual box size=0.8153165213336812 1.0431142960911555 0.12766995280502216
- link Link2: geometry collision box size=0.8600618143328433 0.8293267693940193 0.9678578064494086; visual box size=0.8600618143328433 0.8293267693940193 0.9678578064494086
- link Link3: geometry collision box size=0.6330203075163148 0.48185380233716013 0.13291348360948543; visual box size=0.6330203075163148 0.48185380233716013 0.13291348360948543
- link Link4: geometry collision box size=0.6256443572027992 0.8421034346280386 0.6070166750685325; visual box size=0.6256443572027992 0.8421034346280386 0.6070166750685325
Joints:
- removed joint Link0_Link3
- removed joint Link1_Link2
- removed joint Link1_Link4
- added joint Link0_Link2: type revolute, parent Link0, child Link2, origin xyz=0 0 1.5 rpy=0 0 0, axis 0 0 1, limit lower=-3.14159 upper=3.14159 effort=0.0 velocity=0.0
- added joint Link0_Link6: type revolute, parent Link0, child Link6, origin xyz=0.5 0 1 rpy=0 0 0, axis 0 1 0, limit lower=-3.14159 upper=3.14159 effort=0.0 velocity=0.0
- added joint Link2_Link3: type revolute, parent Link2, child Link3, origin xyz=0 -0.41466338469700964 0 rpy=0 0 0, axis 1 0 0, limit lower=-3.14159 upper=3.14159 effort=0.0 velocity=0.0
- added joint Link3_Link4: type revolute, parent Link3, child Link4, origin xyz=0 0 -0.06645674180474272 rpy=0 0 0, axis 0 0 1, limit lower=-3.14159 upper=3.14159 effort=0.0 velocity=0.0
- added joint Link4_Link5: type revolute, parent Link4, child Link5, origin xyz=0 -0.4210517173140193 0 rpy=0 0 0, axis 1 0 0, limit lower=-3.14159 upper=3.14159 effort=0.0 velocity=0.0
- added joint Link4_Link7: type revolute, parent Link4, child Link7, origin xyz=0 0 -0.30350833753426626 rpy=0 0 0, axis 0 0 1, limit lower=-3.14159 upper=3.14159 effort=0.0 velocity=0.0
- joint Link0_Link1: axis 0 1 0 -> 0 0 1; origin xyz=0.5 0 1 rpy=0 0 0 -> xyz=0 0 0.5 rpy=0 0 0

File: body7.urdf (robot description, URDF)
Before this commit: robot robot, 7 links, 6 joints
Links:
- link Link1: geometry collision box size=0.7581225952937569 0.5334572816580214 0.4158284206448998; visual box size=0.7581225952937569 0.5334572816580214 0.4158284206448998
- link Link2: geometry collision box size=0.6470773191447883 0.9533962707001292 0.26870776421091835; visual box size=0.6470773191447883 0.9533962707001292 0.26870776421091835
- link Link3: geometry collision box size=0.6576919575772031 0.482913586546702 0.8055789418038266; visual box size=0.6576919575772031 0.482913586546702 0.8055789418038266
- link Link4: geometry collision box size=0.540949712924473 0.36954083663878967 0.30366073393483195; visual box size=0.540949712924473 0.36954083663878967 0.30366073393483195
- link Link5: geometry collision box size=0.6717473258068808 0.9392822622987711 0.2100168719993796; visual box size=0.6717473258068808 0.9392822622987711 0.2100168719993796
- link Link6: geometry collision box size=0.12494974408883155 0.9465490839307625 0.4335407364864792; visual box size=0.12494974408883155 0.9465490839307625 0.4335407364864792
Joints:
- removed joint Link0_Link3
- removed joint Link0_Link5
- removed joint Link1_Link2
- removed joint Link3_Link6
- added joint Link0_Link2: type revolute, parent Link0, child Link2, origin xyz=0 0 1.5 rpy=0 0 0, axis 0 0 1, limit lower=-3.14159 upper=3.14159 effort=0.0 velocity=0.0
- added joint Link0_Link6: type revolute, parent Link0, child Link6, origin xyz=0 0 0.5 rpy=0 0 0, axis 0 0 1, limit lower=-3.14159 upper=3.14159 effort=0.0 velocity=0.0
- added joint Link1_Link3: type revolute, parent Link1, child Link3, origin xyz=-0.7581225952937569 0 0 rpy=0 0 0, axis 0 1 0, limit lower=-3.14159 upper=3.14159 effort=0.0 velocity=0.0
- added joint Link1_Link5: type revolute, parent Link1, child Link5, origin xyz=0 0.5334572816580214 0 rpy=0 0 0, axis 1 0 0, limit lower=-3.14159 upper=3.14159 effort=0.0 velocity=0.0
- joint Link0_Link1: axis 0 0 1 -> 0 1 0; origin xyz=0 0 0.5 rpy=0 0 0 -> xyz=0.5 0 1 rpy=0 0 0
- joint Link1_Link4: origin xyz=0 0 0.34424596935082824 rpy=0 0 0 -> xyz=0 0 0.2079142103224499 rpy=0 0 0

File: body8.urdf (robot description, URDF)
Before this commit: robot robot, 7 links, 6 joints
Links:
- added link Link7, mass 1; collision box size=0.45549226736152193 0.658911978719478 0.9610509063492852; visual box size=0.45549226736152193 0.658911978719478 0.9610509063492852
- link Link1: geometry collision box size=0.418754921383494 0.4535787424720895 0.6443214550381721; visual box size=0.418754921383494 0.4535787424720895 0.6443214550381721
- link Link2: geometry collision box size=0.37662331894193923 0.7157448671956707 0.18899039457002045; visual box size=0.37662331894193923 0.7157448671956707 0.18899039457002045
- link Link3: geometry collision box size=0.9901363288852127 1.035055780942857 0.22101429503811745; visual box size=0.9901363288852127 1.035055780942857 0.22101429503811745
- link Link4: geometry collision box size=0.4897814639964124 1.0309561813026746 0.2241574684293636; visual box size=0.4897814639964124 1.0309561813026746 0.2241574684293636
- link Link5: geometry collision box size=1.043944129687256 0.5188515606584863 0.48223452618878904; visual box size=1.043944129687256 0.5188515606584863 0.48223452618878904
- link Link6: geometry collision box size=0.17989275554139886 0.691933858496368 0.17280745799790356; visual box size=0.17989275554139886 0.691933858496368 0.17280745799790356
Joints:
- removed joint Link0_Link6
- removed joint Link4_Link5
- added joint Link2_Link6: type revolute, parent Link2, child Link6, origin xyz=-0.37662331894193923 0 0 rpy=0 0 0, axis 0 1 0, limit lower=-3.14159 upper=3.14159 effort=0.0 velocity=0.0
- added joint Link3_Link5: type revolute, parent Link3, child Link5, origin xyz=0 1.035055780942857 0 rpy=0 0 0, axis 1 0 0, limit lower=-3.14159 upper=3.14159 effort=0.0 velocity=0.0
- added joint Link6_Link7: type revolute, parent Link6, child Link7, origin xyz=0 0 -0.08640372899895178 rpy=0 0 0, axis 0 0 1, limit lower=-3.14159 upper=3.14159 effort=0.0 velocity=0.0
- joint Link0_Link1: axis 1 0 0 -> 0 0 1; origin xyz=0 0.5 1 rpy=0 0 0 -> xyz=0 0 1.5 rpy=0 0 0
- joint Link1_Link2: axis 1 0 0 -> 0 1 0; origin xyz=0 0.7453295674090956 0 rpy=0 0 0 -> xyz=0.418754921383494 0 0 rpy=0 0 0
- joint Link1_Link3: axis 1 0 0 -> 0 1 0; origin xyz=0 0.7453295674090956 0 rpy=0 0 0 -> xyz=0.418754921383494 0 0 rpy=0 0 0
- joint Link3_Link4: axis 0 0 1 -> 0 1 0; origin xyz=0 0 0.31610987396543505 rpy=0 0 0 -> xyz=-0.9901363288852127 0 0 rpy=0 0 0

File: body9.urdf (robot description, URDF)
Before this commit: robot robot, 5 links, 4 joints
Links:
- added link Link5, mass 1; collision box size=0.8124675875953125 0.6154785553284724 0.5423136928231626; visual box size=0.8124675875953125 0.6154785553284724 0.5423136928231626
- link Link1: geometry collision box size=0.648500844201073 0.336504335942426 0.1768324977179835; visual box size=0.648500844201073 0.336504335942426 0.1768324977179835
- link Link2: geometry collision box size=1.0135407297609595 0.3661030640650461 0.42166310260487194; visual box size=1.0135407297609595 0.3661030640650461 0.42166310260487194
- link Link3: geometry collision box size=0.3857095506151792 0.4733346587691296 0.726226126595371; visual box size=0.3857095506151792 0.4733346587691296 0.726226126595371
- link Link4: geometry collision box size=0.1711014253315231 0.16586437433646664 0.8443779112033238; visual box size=0.1711014253315231 0.16586437433646664 0.8443779112033238
Joints:
- removed joint Link1_Link2
- removed joint Link1_Link4
- added joint Link0_Link2: type revolute, parent Link0, child Link2, origin xyz=0 0 0.5 rpy=0 0 0, axis 0 0 1, limit lower=-3.14159 upper=3.14159 effort=0.0 velocity=0.0
- added joint Link0_Link5: type revolute, parent Link0, child Link5, origin xyz=-0.5 0 1 rpy=0 0 0, axis 0 1 0, limit lower=-3.14159 upper=3.14159 effort=0.0 velocity=0.0
- added joint Link2_Link4: type revolute, parent Link2, child Link4, origin xyz=0 0.3661030640650461 0 rpy=0 0 0, axis 1 0 0, limit lower=-3.14159 upper=3.14159 effort=0.0 velocity=0.0
- joint Link0_Link1: axis 1 0 0 -> 0 1 0; origin xyz=0 -0.5 1 rpy=0 0 0 -> xyz=0.5 0 1 rpy=0 0 0
- joint Link0_Link3: axis 1 0 0 -> 0 1 0; origin xyz=0 -0.5 1 rpy=0 0 0 -> xyz=-0.5 0 1 rpy=0 0 0
